File: kicad/diyaltimeter.de.kicad_pcb (KiCad board)
At the start: 2 copper layers, 45.7 x 97.8 mm, 12 parts, among them J1 Buttons, J2 Display, J3 links, J4 rechts, J5 I2C_BMP280, J6 I2C_BMP280_2, J7 RTC DS3231, J8 Conn_01x04_Male, SW1 SW_Push, SW2 SW_Push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

Commit message: pcb re-leayout
Parts:
- moved J2 2.54 mm to (81.3, 109.2)
- moved C1 1.91 mm to (71.1, 120.0)
Routing:
- net SDA: track 24.7 -> 27.2 mm
- net SCL: track 42.4 -> 45.0 mm
- net RES: track 60.5 -> 63.1 mm
- net DC: track 65.6 -> 68.1 mm
- net CS: track 42.0 -> 44.5 mm
- net RS: track 13.0 -> 14.9 mm
- net +3V3: vias 1 -> 0
Other:
- outline, holes or cut-outs redrawn
- board text added: "Marcel Verdult diyaltimeter.de - Rev 1.02"
- board text removed: "Marcel Verdult diyaltimeter.de - Rev 1.01"
Changed lines of the file:
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@@
   (general
     (thickness 1.6)
-    (drawings 48)
-    (tracks 76)
+    (drawings 56)
+    (tracks 79)
     (zones 0)
     (modules 12)
@@
   )
   (module Connector_PinHeader_2.54mm:PinHeader_1x07_P2.54mm_Vertical (layer F.Cu)
-    (at 81.28 111.76 90)
+    (at 81.28 109.22 90)
     (descr "Through hole straight pin header, 1x07, 2.54mm pitch, single row")
     (tags "Through hole pin header THT 1x07 2.54mm single row")
@@
   )
   (module Capacitor_THT:C_Rect_L9.0mm_W4.0mm_P7.50mm_MKT (layer F.Cu)
-    (at 71.12 121.92 90)
+    (at 71.12 120.015 90)
     (descr "C, Rect series, Radial, pin pitch=7.50mm, , length*width=9*4.0mm^2, Capacitor, https://en.tdk.eu/inf/20/20/db/fc_2009/MKT_B32560_564.pdf")
     (tags "C Rect series Radial pin pitch 7.50mm  length 9mm width 4.0mm Capacitor")
@@
     (arrow2b (pts (xy 121.92 82.55) (xy 122.506421 83.676504)))
   )
+  (gr_arc (start 68.58 101.6) (end 66.04 101.6) (angle -90) (layer Edge.Cuts) (width 0.05))
+  (gr_arc (start 68.58 85.09) (end 68.58 82.55) (angle -90) (layer Edge.Cuts) (width 0.05))
+  (gr_arc (start 109.22 85.09) (end 111.76 85.09) (angle -90) (layer Edge.Cuts) (width 0.05))
+  (gr_arc (start 109.22 101.6) (end 109.22 104.14) (angle -90) (layer Edge.Cuts) (width 0.05))
+  (gr_line (start 111.76 109.22) (end 111.76 177.8) (layer Edge.Cuts) (width 0.05))
+  (gr_arc (start 109.22 177.8) (end 109.22 180.34) (angle -90) (layer Edge.Cuts) (width 0.05))
+  (gr_arc (start 68.58 177.8) (end 66.04 177.8) (angle -90) (layer Edge.Cuts) (width 0.05))
+  (gr_line (start 68.58 106.68) (end 109.22 106.68) (layer Edge.Cuts) (width 0.05))
+  (gr_arc (start 68.58 109.22) (end 68.58 106.68) (angle -90) (layer Edge.Cuts) (width 0.05))
+  (gr_arc (start 109.22 109.22) (end 111.76 109.22) (angle -90) (layer Edge.Cuts) (width 0.05))
   (gr_text B3 (at 78.74 103.505) (layer F.SilkS)
     (effects (font (size 1 1) (thickness 0.15)))
@@
     (arrow2b (pts (xy 111.76 69.85) (xy 110.633496 70.436421)))
   )
-  (gr_line (start 111.76 104.14) (end 66.04 104.14) (layer Edge.Cuts) (width 0.1))
-  (gr_line (start 111.76 82.55) (end 111.76 104.14) (layer Edge.Cuts) (width 0.1))
-  (gr_line (start 66.04 82.55) (end 111.76 82.55) (layer Edge.Cuts) (width 0.1))
-  (gr_line (start 66.04 104.14) (end 66.04 82.55) (layer Edge.Cuts) (width 0.1))
-  (gr_line (start 111.76 106.68) (end 66.04 106.68) (layer Edge.Cuts) (width 0.1))
-  (gr_line (start 111.76 180.34) (end 111.76 106.68) (layer Edge.Cuts) (width 0.1))
-  (gr_line (start 66.04 180.34) (end 111.76 180.34) (layer Edge.Cuts) (width 0.1))
-  (gr_line (start 66.04 106.68) (end 66.04 180.34) (layer Edge.Cuts) (width 0.1))
+  (gr_line (start 109.22 104.14) (end 68.58 104.14) (layer Edge.Cuts) (width 0.1))
+  (gr_line (start 111.76 85.09) (end 111.76 101.6) (layer Edge.Cuts) (width 0.1))
+  (gr_line (start 68.58 82.55) (end 109.22 82.55) (layer Edge.Cuts) (width 0.1))
+  (gr_line (start 66.04 101.6) (end 66.04 85.09) (layer Edge.Cuts) (width 0.1))
+  (gr_line (start 68.58 180.34) (end 109.22 180.34) (layer Edge.Cuts) (width 0.1))
+  (gr_line (start 66.04 109.22) (end 66.04 177.8) (layer Edge.Cuts) (width 0.1))
   (dimension 45.72 (width 0.12) (layer F.SilkS)
     (gr_text "45,720 mm" (at 88.9 191.77) (layer F.SilkS)
@@
     (arrow2b (pts (xy 66.04 190.5) (xy 67.166504 189.913579)))
   )
-  (gr_text 1uF (at 71.12 124.46) (layer F.SilkS)
-    (effects (font (size 1 1) (thickness 0.15)))
+  (gr_text 1uF (at 71.12 114.3 90) (layer F.SilkS)
+    (effects (font (size 1 1) (thickness 0.15)) (justify right))
   )
   (gr_text BMP280 (at 99.06 144.78) (layer F.SilkS)
@@
     (effects (font (size 1 1) (thickness 0.15)))
   )
-  (gr_text "Marcel Verdult\ndiyaltimeter.de - Rev 1.01" (at 107.95 119.38 90) (layer F.SilkS)
+  (gr_text "Marcel Verdult\ndiyaltimeter.de - Rev 1.02" (at 109.22 121.92 90) (layer F.SilkS)
     (effects (font (size 1 1) (thickness 0.15)))
   )
@@
   (segment (start 78.74 139.7) (end 71.12 147.32) (width 0.8) (layer F.Cu) (net 3))
   (segment (start 78.74 109.22) (end 78.74 139.7) (width 0.8) (layer F.Cu) (net 3))
-  (segment (start 83.82 111.76) (end 83.82 111.76) (width 0.8) (layer F.Cu) (net 5))
-  (via (at 83.82 111.76) (size 0.8) (drill 0.4) (layers F.Cu B.Cu) (net 5))
   (segment (start 93.98 147.32) (end 87.63 147.32) (width 0.8) (layer F.Cu) (net 6))
   (segment (start 87.63 147.32) (end 86.36 146.05) (width 0.8) (layer F.Cu) (net 6))
   (segment (start 86.36 146.05) (end 86.36 111.76) (width 0.8) (layer F.Cu) (net 6))
+  (segment (start 86.36 111.76) (end 86.36 109.22) (width 0.8) (layer F.Cu) (net 6))
   (segment (start 88.9 111.76) (end 88.9 130.81) (width 0.8) (layer F.Cu) (net 7))
   (segment (start 88.9 130.81) (end 90.17 132.08) (width 0.8) (layer F.Cu) (net 7))
   (segment (start 90.17 132.08) (end 93.98 132.08) (width 0.8) (layer F.Cu) (net 7))
+  (segment (start 88.9 111.76) (end 88.9 109.22) (width 0.8) (layer F.Cu) (net 7))
   (segment (start 91.44 111.76) (end 91.44 121.92) (width 0.8) (layer B.Cu) (net 8))
   (segment (start 91.44 121.92) (end 87.63 125.73) (width 0.8) (layer B.Cu) (net 8))
@@
   (segment (start 87.63 153.67) (end 86.36 154.94) (width 0.8) (layer B.Cu) (net 8))
   (segment (start 86.36 154.94) (end 71.12 154.94) (width 0.8) (layer B.Cu) (net 8))
+  (segment (start 91.44 111.76) (end 91.44 109.22) (width 0.8) (layer B.Cu) (net 8))
   (segment (start 71.12 157.48) (end 88.9 157.48) (width 0.8) (layer B.Cu) (net 9))
   (segment (start 88.9 157.48) (end 90.17 156.21) (width 0.8) (layer B.Cu) (net 9))
@@
   (segment (start 93.98 123.19) (end 93.98 111.76) (width 0.8) (layer B.Cu) (net 9))
   (segment (start 90.17 127) (end 93.98 123.19) (width 0.8) (layer B.Cu) (net 9))
+  (segment (start 93.98 111.76) (end 93.98 109.22) (width 0.8) (layer B.Cu) (net 9))
   (segment (start 96.52 111.76) (end 96.52 124.46) (width 0.8) (layer B.Cu) (net 10))
   (segment (start 96.52 124.46) (end 93.98 127) (width 0.8) (layer B.Cu) (net 10))
@@
   (segment (start 91.44 147.32) (end 93.98 149.86) (width 0.8) (layer B.Cu) (net 10))
   (segment (start 91.44 128.27) (end 91.44 147.32) (width 0.8) (layer B.Cu) (net 10))
-  (segment (start 71.12 121.92) (end 68.58 124.46) (width 0.8) (layer F.Cu) (net 11))
-  (segment (start 68.58 124.46) (end 68.58 130.81) (width 0.8) (layer F.Cu) (net 11))
-  (segment (start 68.58 130.81) (end 69.85 132.08) (width 0.8) (layer F.Cu) (net 11))
-  (segment (start 69.85 132.08) (end 71.12 132.08) (width 0.8) (layer F.Cu) (net 11))
+  (segment (start 96.52 111.76) (end 96.52 109.22) (width 0.8) (layer B.Cu) (net 10))
+  (segment (start 68.58 122.555) (end 71.12 120.015) (width 0.8) (layer F.Cu) (net 11))
+  (segment (start 68.58 130.81) (end 68.58 122.555) (width 0.8) (layer F.Cu) (net 11))
+  (segment (start 71.12 132.08) (end 69.85 132.08) (width 0.8) (layer F.Cu) (net 11))
+  (segment (start 69.85 132.08) (end 68.58 130.81) (width 0.8) (layer F.Cu) (net 11))
   (segment (start 99.06 152.4) (end 100.33 152.4) (width 0.8) (layer F.Cu) (net 21))
   (segment (start 100.33 152.4) (end 101.6 151.13) (width 0.8) (layer F.Cu) (net 21))
@@
   (segment (start 71.12 101.6) (end 71.12 98.9464) (width 0.8) (layer F.Cu) (net 39))
   (segment (start 73.74 97.59) (end 73.74 85.09) (width 0.8) (layer F.Cu) (net 39))
-  (zone (net 38) (net_name "Net-(J8-Pad3)") (layer B.Cu) (hatch edge 0.508)
-    (connect_pads (clearance 0.508))
-    (min_thickness 0.254)
-    (fill yes (arc_segments 32) (thermal_gap 0.508) (thermal_bridge_width 0.508))
-    (polygon
-      (pts
-        (xy 66.04 82.55) (xy 66.04 104.14) (xy 111.76 104.14) (xy 111.76 82.55)
-      )
-    )
-  )
   (zone (net 4) (net_name GND) (layer F.Cu) (hatch edge 0.508)
     (connect_pads (clearance 0.508))
@@
       )
     )
+  )
+  (zone (net 38) (net_name "Net-(J8-Pad3)") (layer B.Cu) (hatch edge 0.508)
+    (connect_pads (clearance 0.508))
+    (min_thickness 0.254)
+    (fill yes (arc_segments 32) (thermal_gap 0.508) (thermal_bridge_width 0.508))
+    (polygon
+      (pts
+        (xy 66.04 81.28) (xy 66.04 104.14) (xy 111.76 104.14) (xy 111.76 81.28)
+      )
+    )

Commit message: final pcb
Parts:
- added C2: C, Capacitor_SMD:C_0805_2012Metric_Pad1.15x1.40mm_HandSolder, F.Cu at (71.1, 116.2)
Routing:
- net RS: track 14.9 -> 17.7 mm
